File: CoaxTestAdapter.kicad_sch (KiCad schematic)
At the start: 7 parts, among them J1 Conn_Coaxial, J2 Conn_Coaxial, J3 Conn_01x01_Socket, J4 Conn_01x01_Socket, SW1 SW_Push_DPDT, SW2 SW_Push_DPDT, SW3 SW_Push_Open

Commit message: guh
Parts:
- removed SW1, SW2: SW_Push_DPDT, symbol Switch:SW_Push_DPDT
- removed SW3: SW_Push_Open, symbol Switch:SW_Push_Open
- added H1, H2: M3, MountingHole:MountingHole_3.2mm_M3_DIN965, symbol Mechanical:MountingHole
- added SW1: MRK403-A, Library:MRK403-A_NKK, symbol New_Library:MRK403-A
- J1, J2: value Conn_Coaxial -> 0731000154; footprint (none) -> Library:0731000154
- J3, J4: value Conn_01x01_Socket -> 72918; footprint (none) -> MountingHole:MountingHole_3.2mm_M3_DIN965_Pad
Connections:
- net C2: now reaches J2.1 (In)
- net C2: now also SW1.13
- net S2: now reaches J2.2 (Ext)
- net S2: now also SW1.9
- net C1: now reaches J1.1 (In)
- net C1: now also SW1.5
- net O1: now reaches J3.1 (Pin_1)
- net O1: now also SW1.3, SW1.6, SW1.8
- net O2: now reaches J4.1 (Pin_1)
- net O2: now also SW1.11, SW1.12, SW1.14
- net s1 renamed S1
- net S1: now also SW1.1
- no-connect marks 0 -> 6
Other:
- note added: "TEST A"
- note added: "TEST A Connects C1 to C2, testing center continuity. TEST B Connects S1 to S2, testing shield continuity. TEST C Connects C1 to S2, testing cross conductor shorts."
- note added: "TEST B"
- note added: "TEST C"
- note removed: "100-dp1-t1-b1-m1-q-e-h: DPDT on-none-on"
- moved on the sheet: J1, J3, J4
